File: Hardware/PCB/ExpansionBoard/Airspeed.kicad_sch (KiCad schematic)
At the start: 0 parts

Commit message: finished schema
Parts:
- added Air601: 4525DO-DS5AI015DP, DynamicSoaring:4525DO-DS5AI015DP, symbol DynamicSoaring:4525DO-DS5AI015DP
- added C601: 100n, Capacitor_SMD:C_0805_2012Metric_Pad1.18x1.45mm_HandSolder, symbol Device:C_Small
Connections:
- new net: Air601.6 (NC1), Air601.7 (NC2), Air601.8 (NC3)
- new net +3.3V: Air601.2 (VCC), C601.1
- new net GND: Air601.1 (GND), C601.2
- new net INT: Air601.5 (INT)
- new net SCL: Air601.4 (SCL/SCLK)
- new net SDA: Air601.3 (SDA/MISO)
