File: Hardware/PCB/ExpansionBoard/MCU.kicad_sch (KiCad schematic)
At the start: 25 parts, among them IC301 STM32L452RET6, J301 ResertConnector, J302 Conn_01x06_Socket, J303 MEM2061-01-188-00-A

Commit message: finished pcb layout
Parts:
- IC301: footprint SamacSys_Parts:QFP50P1200X1200X160-64N -> QFP50P1200X1200X160-64N
- J303: footprint SamacSys_Parts:MEM20610118800A -> MEM20610118800A
Connections:
- net MISO: no longer IC301.10 (PC2), J303.P7 (DAT0)
- net MOSI: no longer IC301.11 (PC3), J303.P3 (CMD)
- net CLK renamed SD_CLK
- net NSS renamed SD_NSS
- new net SD_MISO: IC301.10 (PC2), J303.P7 (DAT0)
- new net SD_MOSI: IC301.11 (PC3), J303.P3 (CMD)
Changed lines of the file:
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@@
 	(paper "A4")
 	(bus_alias "SD_Card"
-		(members "NSS" "MOSI" "MISO" "CLK" "CardDetect")
+		(members "SD_NSS" "SD_MOSI" "SD_MISO" "SD_CLK" "CardDetect")
 	)
 	(bus_alias "UART"
@@
 		)
 	)
-	(label "MISO"
+	(label "SD_MISO"
 		(at 87.63 118.11 0)
+		(fields_autoplaced yes)
 		(effects
 			(font
@@
 		)
 	)
-	(label "MISO"
+	(label "SD_MISO"
 		(at 240.03 121.92 90)
+		(fields_autoplaced yes)
 		(effects
 			(font
@@
 		)
 	)
-	(label "CLK"
+	(label "SD_CLK"
 		(at 138.43 160.02 90)
+		(fields_autoplaced yes)
 		(effects
 			(font
@@
 		)
 	)
-	(label "CLK"
+	(label "SD_CLK"
 		(at 245.11 121.92 90)
+		(fields_autoplaced yes)
 		(effects
 			(font
@@
 	(label "CardDetect"
 		(at 115.57 58.42 90)
+		(fields_autoplaced yes)
 		(effects
 			(font
@@
 	(label "CardDetect"
 		(at 232.41 121.92 180)
+		(fields_autoplaced yes)
 		(effects
 			(font
@@
 		)
 	)
-	(label "MOSI"
+	(label "SD_MOSI"
 		(at 87.63 120.65 0)
+		(fields_autoplaced yes)
 		(effects
 			(font
@@
 		)
 	)
-	(label "NSS"
+	(label "SD_NSS"
 		(at 105.41 46.99 180)
+		(fields_autoplaced yes)
 		(effects
 			(font
@@
 		)
 	)
-	(label "MOSI"
+	(label "SD_MOSI"
 		(at 234.95 64.77 90)
+		(fields_autoplaced yes)
 		(effects
 			(font
@@
 		)
 	)
-	(label "NSS"
+	(label "SD_NSS"
 		(at 237.49 64.77 90)
+		(fields_autoplaced yes)
 		(effects
 			(font
@@
 			)
 		)
-		(property "Footprint" "SamacSys_Parts:QFP50P1200X1200X160-64N"
+		(property "Footprint" "QFP50P1200X1200X160-64N"
 			(at 157.48 162.23 0)
 			(effects
@@
 			)
 		)
-		(property "Footprint" "SamacSys_Parts:MEM20610118800A"
+		(property "Footprint" "MEM20610118800A"
 			(at 150.19 107.95 0)
 			(effects

Commit message: finsihed pcb
Parts:
- IC301: footprint QFP50P1200X1200X160-64N -> SamacSys_Parts:QFP50P1200X1200X160-64N
- J303: footprint MEM20610118800A -> SamacSys_Parts:MEM20610118800A
Changed lines of the file:
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@@
 			)
 		)
-		(property "Footprint" "QFP50P1200X1200X160-64N"
+		(property "Footprint" "SamacSys_Parts:QFP50P1200X1200X160-64N"
 			(at 157.48 162.23 0)
 			(effects
@@
 			)
 		)
-		(property "Footprint" "MEM20610118800A"
+		(property "Footprint" "SamacSys_Parts:MEM20610118800A"
 			(at 150.19 107.95 0)
 			(effects
