File: Hardware/PCB/ExpansionBoard/UART_USB.kicad_sch (KiCad schematic)
At the start: 2 parts, among them J501 USB_B_Micro, U501 FT232RL

Commit message: added USB and Powerseitcher
Parts:
- added C501: 4.7u, symbol Device:C_Polarized_Small
- added C502, C503, C504: 47p, symbol Device:C_Small
- added C505, C506, C508: 0.1u, symbol Device:C_Small
- added C507: 10n, symbol Device:C_Polarized_Small
- added FB501: FerriteBead, symbol Device:FerriteBead
- added JP501, JP502: SolderJumper_2_Open, symbol Jumper:SolderJumper_2_Open
- added R501: 0, symbol Device:R_Small
- added R502: DO NOT CONNECT, symbol Device:R_Small
Connections:
- net GND: now also J501.5 (GND), J501.6 (Shield), C501.2, C502.2, C503.2, C504.2, C505.1, C506.2, C507.2, JP501.1 (A), R501.2
- net MCU_RX: now reaches U501.1 (TXD)
- net MCU_RTS: now reaches U501.11 (CTS)
- net at U501.15 (USBD+): now also J501.3 (D+)
- net at U501.16 (USBD-): now also J501.2 (D-)
- net at U501.17 (3V3OUT): now also C505.2
- net +5V: now reaches U501.20 (VCC)
- net +5V: now also C501.1, C502.1, C503.1, C504.1, C506.1, C507.1, FB501.2
- net MCU_CTS: now reaches U501.3 (RTS)
- net at U501.4 (VCCIO): now also C508.2
- net MCU_TX: now reaches U501.5 (RXD)
- net at J501.1 (VBUS): now also FB501.1
- net at J501.4 (ID): now also R501.1, R502.1
- new net: JP501.2 (B), JP502.2 (B), R502.2
- new net +3.3V: C508.1, JP502.1 (A)
Other:
- moved on the sheet: J501

Commit message: DONE: PWR LED MISSING AND AIRSPEED
Parts:
- added D501: LED BLAU, symbol Device:LED
- added D502: LED Orange, symbol Device:LED
- added R503: 20, symbol Device:R_Small
- added R504: 56, symbol Device:R_Small
- added TP501, TP502, TP503, TP504, TP505, TP506, TP507, TP508, TP509, TP510: TestPoint, symbol Connector:TestPoint
Connections:
- net +3.3V: now also U501.4 (VCCIO), D501.2 (A), D502.2 (A)
- net GND: now also C508.2
- net at U501.10 (DCD): now also TP503.1
- net at U501.12 (CBUS4): now also TP507.1
- net at U501.13 (CBUS2): now also TP505.1
- net at U501.14 (CBUS3): now also TP506.1
- net at U501.19 (~{RESET}): now also TP510.1
- net at U501.2 (DTR): now also TP501.1
- net at U501.22 (CBUS1): now also R504.1
- net at U501.23 (CBUS0): now also R503.1
- net at U501.27 (OSCI): now also TP509.1
- net at U501.28 (OSCO): now also TP508.1
- net at U501.6 (RI): now also TP504.1
- net at U501.9 (DCR): now also TP502.1
- new net: D502.1 (K), R504.2
- new net: D501.1 (K), R503.2
Other:
- moved on the sheet: C508

Commit message: finished schema
Parts:
- removed J501: USB_B_Micro, symbol Connector:USB_B_Micro
- added J502: 2173157-3, 21731573, symbol SamacSys_Parts:2173157-3
- C501, C502, C503, C504, C505, C506, C507, C508, FB501: footprint (none) -> Capacitor_SMD:C_0805_2012Metric_Pad1.18x1.45mm_HandSolder
- D501: footprint (none) -> SamacSys_Parts:LEDM2012X100N
- D502: footprint (none) -> Resistor_SMD:R_0805_2012Metric
- JP501, JP502: footprint (none) -> Jumper:SolderJumper-2_P1.3mm_Open_RoundedPad1.0x1.5mm
- R501, R502, R503, R504: footprint (none) -> Resistor_SMD:R_0805_2012Metric_Pad1.20x1.40mm_HandSolder
- TP501, TP502, TP503, TP504, TP505, TP506, TP507, TP508, TP509, TP510: footprint (none) -> TestPoint:TestPoint_Pad_D3.0mm
Connections:
- net GND: now also J502.5 (GND), J502.MP1, J502.MP2, J502.MP3, J502.MP4
- net at FB501.1: now also J502.1 (VBUS)
- net at U501.15 (USBD+): now also J502.3 (D+)
- net at U501.16 (USBD-): now also J502.2 (D-)
- net at R501.1, R502.1: now also J502.4 (ID)

Commit message: to pcb
Parts:
- J502: footprint 21731573 -> SamacSys_Parts:21731573
- TP501, TP502, TP503, TP504, TP505, TP506, TP507, TP508, TP509, TP510: footprint TestPoint:TestPoint_Pad_D3.0mm -> TestPoint:TestPoint_Pad_D1.5mm
- U501: symbol Interface_USB:FT232RL -> DynamicSoaring:FT232RL_Fabian
Connections:
- new net: U501.24 (NC), U501.8 (NC)
Changed lines of the file:
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@@
 			)
 		)
-		(property "Footprint" "TestPoint:TestPoint_Pad_D3.0mm"
+		(property "Footprint" "TestPoint:TestPoint_Pad_D1.5mm"
 			(at 182.88 101.6 0)
 			(effects
@@
 			)
 		)
-		(property "Footprint" "TestPoint:TestPoint_Pad_D3.0mm"
+		(property "Footprint" "TestPoint:TestPoint_Pad_D1.5mm"
 			(at 182.88 99.06 0)
 			(effects
@@
 			)
 		)
-		(property "Footprint" "TestPoint:TestPoint_Pad_D3.0mm"
+		(property "Footprint" "TestPoint:TestPoint_Pad_D1.5mm"
 			(at 182.88 86.36 0)
 			(effects
@@
 			)
 		)
-		(property "Footprint" "TestPoint:TestPoint_Pad_D3.0mm"
+		(property "Footprint" "TestPoint:TestPoint_Pad_D1.5mm"
 			(at 182.88 83.82 0)
 			(effects
@@
 			)
 		)
-		(property "Footprint" "TestPoint:TestPoint_Pad_D3.0mm"
+		(property "Footprint" "TestPoint:TestPoint_Pad_D1.5mm"
 			(at 182.88 78.74 0)
 			(effects
@@
 			)
 		)
-		(property "Footprint" "TestPoint:TestPoint_Pad_D3.0mm"
+		(property "Footprint" "TestPoint:TestPoint_Pad_D1.5mm"
 			(at 182.88 81.28 0)
 			(effects
@@
 			)
 		)
-		(property "Footprint" "21731573"
+		(property "Footprint" "SamacSys_Parts:21731573"
 			(at 55.88 158.42 0)
 			(effects
@@
 	)
 	(symbol
-		(lib_id "Interface_USB:FT232RL")
+		(lib_id "DynamicSoaring:FT232RL_Fabian")
 		(at 158.75 81.28 0)
 		(unit 1)
@@
 		(pin "21"
 		)
+		(pin "8"
+		)
+		(pin "24"
+		)
 		(instances
 			(project ""
@@
 			)
 		)
-		(property "Footprint" "TestPoint:TestPoint_Pad_D3.0mm"
+		(property "Footprint" "TestPoint:TestPoint_Pad_D1.5mm"
 			(at 134.62 76.2 0)
 			(effects
@@
 			)
 		)
-		(property "Footprint" "TestPoint:TestPoint_Pad_D3.0mm"
+		(property "Footprint" "TestPoint:TestPoint_Pad_D1.5mm"
 			(at 134.62 86.36 0)
 			(effects
@@
 			)
 		)
-		(property "Footprint" "TestPoint:TestPoint_Pad_D3.0mm"
+		(property "Footprint" "TestPoint:TestPoint_Pad_D1.5mm"
 			(at 182.88 104.14 0)
 			(effects
@@
 			)
 		)
-		(property "Footprint" "TestPoint:TestPoint_Pad_D3.0mm"
+		(property "Footprint" "TestPoint:TestPoint_Pad_D1.5mm"
 			(at 134.62 81.28 0)
 			(effects

Commit message: finished pcb layout
Parts:
- J502: footprint SamacSys_Parts:21731573 -> 21731573
Changed lines of the file:
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@@
 			)
 		)
-		(property "Footprint" "SamacSys_Parts:21731573"
+		(property "Footprint" "21731573"
 			(at 55.88 158.42 0)
 			(effects

Commit message: finsihed pcb
Parts:
- J502: footprint 21731573 -> SamacSys_Parts:21731573
Changed lines of the file:
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@@
 			)
 		)
-		(property "Footprint" "21731573"
+		(property "Footprint" "SamacSys_Parts:21731573"
 			(at 55.88 158.42 0)
 			(effects
